File: pcb/matrix.sch (KiCad schematic (older format))
At the start: 86 parts, among them SW10 SW_PUSH, SW11 SW_PUSH, SW12 SW_PUSH, SW13 SW_PUSH, SW14 SW_PUSH, SW15 SW_PUSH, SW16 SW_PUSH, SW17 SW_PUSH, SW18 SW_PUSH, SW19 SW_PUSH, SW2 SW_PUSH, SW20 SW_PUSH, SW21 SW_PUSH, SW22 SW_PUSH, SW23 SW_PUSH, SW24 SW_PUSH, SW25 SW_PUSH, SW26 SW_PUSH, SW27 SW_PUSH, SW28 SW_PUSH, SW29 SW_PUSH, SW3 SW_PUSH, SW30 SW_PUSH, SW31 SW_PUSH, SW32 SW_PUSH, SW33 SW_PUSH, SW34 SW_PUSH, SW35 SW_PUSH, SW36 SW_PUSH, SW37 SW_PUSH, SW38 SW_PUSH, SW39 SW_PUSH, SW4 SW_PUSH, SW40 SW_PUSH, SW41 SW_PUSH, SW42 SW_PUSH, SW43 SW_PUSH, SW44 SW_PUSH, SW5 SW_PUSH, SW6 SW_PUSH, SW7 SW_PUSH, SW8 SW_PUSH, SW9 SW_PUSH

Commit message: Routing
Connections:
- net row1: now also D14.1 (K), D16.1 (K), D17.1 (K), D19.1 (K), D22.1 (K)
- net row2: now also D29.1 (K)
Changed lines of the file:
@@
 	6525 2625 6525 2690
-$Comp
-L Device:D D19
-U 1 1 5E1853A5
-P 6525 2840
-F 0 "D19" V 6571 2761 50  0000 R CNN
-F 1 "D" V 6480 2761 50  0000 R CNN
-F 2 "Diode_SMD:D_SOD-123" H 6525 2840 50  0001 C CNN
-F 3 "~" H 6525 2840 50  0001 C CNN
-	1    6525 2840
-	0    -1   -1   0
-$EndComp
 $Comp
 L kbd:SW_PUSH SW20
@@
 Wire Wire Line
 	5925 3165 5925 3755
-Connection ~ 5795 2990
 Connection ~ 5795 3530
 Wire Wire Line
@@
 	3515 1995 3515 2625
 Connection ~ 3515 2625
-Wire Wire Line
-	1520 2990 3225 2990
 Connection ~ 3225 2990
-Wire Wire Line
-	3225 2990 5795 2990
-Wire Wire Line
-	8190 2990 9775 2990
 Connection ~ 9775 2990
 Wire Wire Line
@@
 	7380 3530 8190 3530
 Wire Wire Line
-	5795 2990 7380 2990
-Connection ~ 7380 2990
-Wire Wire Line
 	7380 2990 8190 2990
 Connection ~ 7590 3165
@@
 	4290 3165 4290 3755
 Connection ~ 4115 3530
-Wire Wire Line
-	4115 3530 5795 3530
 Wire Wire Line
 	3515 2625 3515 3165
@@
 Text GLabel 800  2360 0    50   Input ~ 0
 row0
+Connection ~ 7380 2990
+Connection ~ 5795 2990
+Wire Wire Line
+	5795 2990 6525 2990
+$Comp
+L Device:D D19
+U 1 1 5E1853A5
+P 6525 2840
+F 0 "D19" V 6571 2761 50  0000 R CNN
+F 1 "D" V 6480 2761 50  0000 R CNN
+F 2 "Diode_SMD:D_SOD-123" H 6525 2840 50  0001 C CNN
+F 3 "~" H 6525 2840 50  0001 C CNN
+	1    6525 2840
+	0    -1   -1   0
+$EndComp
+Wire Wire Line
+	6525 2990 6525 2995
+Connection ~ 6525 2990
+Wire Wire Line
+	6525 2990 7380 2990
+Wire Wire Line
+	8190 2990 8985 2990
+Connection ~ 8985 2990
+Wire Wire Line
+	8985 2990 9775 2990
+Connection ~ 4890 2990
+Wire Wire Line
+	4890 2990 5795 2990
+Wire Wire Line
+	3225 2990 4115 2990
+Connection ~ 4115 2990
+Wire Wire Line
+	4115 2990 4890 2990
+Wire Wire Line
+	1520 2990 2415 2990
+Connection ~ 2415 2990
+Wire Wire Line
+	2415 2990 3225 2990
+Wire Wire Line
+	4115 3530 4890 3530
+Connection ~ 4890 3530
+Wire Wire Line
+	4890 3530 5795 3530
 $EndSCHEMATC

Commit message: fix dcr check error and chgenge switch footprint
Parts:
- SW10, SW11, SW12, SW13, SW14, SW15, SW16, SW17, SW18, SW19, SW2, SW20, SW21, SW22, SW23, SW24, SW25, SW26, SW27, SW28, SW29, SW3, SW30, SW31, SW32, SW33, SW34, SW35, SW36, SW37, SW38, SW39, SW4, SW41, SW43, SW44, SW5, SW6, SW7, SW8, SW9: footprint kbd:CherryMX-Hotswap-v2 -> MX_Only:MXOnly-1U-Hotswap
- SW40, SW42: footprint kbd:CherryMX-Hotswap-v2 -> MX_Only:MXOnly-1.5U-Hotswap
