File: pcb/psykbd.kicad_pcb (KiCad board)
At the start: 2 copper layers, 263.2 x 90.2 mm, 102 parts, among them SW1 SW_PUSH, SW10 SW_PUSH, SW11 SW_PUSH, SW12 SW_PUSH, SW13 SW_PUSH, SW14 SW_PUSH, SW15 SW_PUSH, SW16 SW_PUSH, SW17 SW_PUSH, SW18 SW_PUSH, SW19 SW_PUSH, SW2 SW_PUSH, SW20 SW_PUSH, SW21 SW_PUSH, SW22 SW_PUSH, SW23 SW_PUSH, SW24 SW_PUSH, SW25 SW_PUSH, SW26 SW_PUSH, SW27 SW_PUSH, SW28 SW_PUSH, SW29 SW_PUSH, SW3 SW_PUSH, SW30 SW_PUSH, SW31 SW_PUSH, SW32 SW_PUSH, SW33 SW_PUSH, SW34 SW_PUSH, SW35 SW_PUSH, SW36 SW_PUSH, SW37 SW_PUSH, SW38 SW_PUSH, SW39 SW_PUSH, SW4 SW_PUSH, SW40 SW_PUSH, SW41 SW_PUSH, SW42 SW_PUSH, SW43 SW_PUSH, SW44 SW_PUSH, SW5 SW_PUSH, SW6 SW_PUSH, SW7 SW_PUSH, SW8 SW_PUSH, SW9 SW_PUSH, U1 ATmega32U4-AU, Y1 16MHz

Commit message: Routing
Parts:
- moved D27 41.4 mm to (240.5, 98.4)
- moved R4 40.9 mm to (162.7, 87.3), turned to 90 degrees
- moved D37 40.2 mm to (221.5, 117.5)
- moved C4 39.5 mm to (140.5, 86.5), turned to 270 degrees
- moved C3 38.8 mm to (140.5, 80.7), turned to 270 degrees
- moved SW38 38.8 mm to (213.5, 117.5)
- moved D39 38.2 mm to (178.6, 117.5)
- moved D38 37.9 mm to (202.4, 117.5)
- moved SW39 37.5 mm to (194.5, 117.5)
- moved SW40 36.8 mm to (170.7, 117.5)
- moved D26 36.2 mm to (259.6, 103.2)
- moved D40 35.8 mm to (159.5, 98.5)
- moved SW28 35.6 mm to (232.6, 98.4)
- moved SW41 33.4 mm to (151.5, 98.4)
- moved D25 33.1 mm to (278.6, 103.2)
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Connections:
- D14 pad 1: Net-(D14-Pad1) -> row1
- D16 pad 1: Net-(D16-Pad1) -> row1
- D17 pad 1: Net-(D17-Pad1) -> row1
- D19 pad 1: Net-(D19-Pad1) -> row1
- D22 pad 1: Net-(D22-Pad1) -> row1
- D29 pad 1: Net-(D29-Pad1) -> row2
- U1 pad 1: Net-(U1-Pad1) -> col11
- U1 pad 10: Net-(U1-Pad10) -> col9
- U1 pad 11: Net-(U1-Pad11) -> col10
- U1 pad 18: Net-(U1-Pad18) -> row0
- U1 pad 19: Net-(U1-Pad19) -> row1
- U1 pad 25: Net-(U1-Pad25) -> col0
- U1 pad 26: Net-(U1-Pad26) -> col1
- U1 pad 27: Net-(U1-Pad27) -> col2
- U1 pad 28: Net-(U1-Pad28) -> col3
- U1 pad 29: Net-(U1-Pad29) -> col4
- U1 pad 30: Net-(U1-Pad30) -> col5
- U1 pad 32: Net-(U1-Pad32) -> col6
- U1 pad 36: Net-(U1-Pad36) -> row3
- U1 pad 37: Net-(U1-Pad37) -> row2
- U1 pad 8: Net-(U1-Pad8) -> col7
- U1 pad 9: Net-(U1-Pad9) -> col8
Routing:
- net row0: track 0.00 -> 200.4 mm
- net row2: track 0.00 -> 200.2 mm
- net row1: track 0.00 -> 200.1 mm
- net row3: track 0.00 -> 148.5 mm
- net GND: track 0.00 -> 20.6 mm
- net VCC: track 0.00 -> 11.5 mm
- net D-: track 0.00 -> 6.47 mm
- net D+: track 0.00 -> 6.32 mm
- net Net-(D35-Pad2): track 0.00 -> 3.66 mm
- net Net-(D36-Pad2): track 0.00 -> 3.59 mm
- net Net-(D24-Pad2): track 0.00 -> 3.59 mm
- net Net-(D23-Pad2): track 0.00 -> 3.59 mm
- net Net-(C2-Pad1): track 0.00 -> 3.36 mm
- net Net-(C1-Pad1): track 0.00 -> 3.36 mm
- net Net-(D40-Pad2): track 0.00 -> 2.89 mm
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Other:
- outline, holes or cut-outs redrawn
- net class class1 added: clearance 0.4, trace_width 0.5, via_dia 0.8, via_drill 0.4

Commit message: chenge mcu position
Parts:
- SW1: moved to B.Cu
- moved C3 13.6 mm to (143.7, 67.5), turned to 180 degrees
- moved R4 7.98 mm to (154.8, 86.5), turned to 0 degrees
- moved C2 7.49 mm to (156.4, 56.4), turned to 180 degrees
- moved C1 6.40 mm to (156.4, 65.9), turned to 0 degrees
- moved C4 6.35 mm to (146.8, 86.5), turned to 180 degrees
- moved F1 5.61 mm to (144.5, 55.6)
- moved U1 4.99 mm to (150.8, 75.4), turned to 315 degrees
- moved R1 2.36 mm to (160.3, 53.2), turned to 0 degrees
- moved Y1 1.77 mm to (156.4, 61.1), turned to 90 degrees
- moved C5 1.59 mm to (161.9, 73.0)
Connections:
- U1 pad 1: col11 -> Net-(U1-Pad1)
- U1 pad 10: col9 -> Net-(U1-Pad10)
- U1 pad 11: col10 -> Net-(U1-Pad11)
- U1 pad 18: row0 -> Net-(U1-Pad18)
- U1 pad 19: row1 -> Net-(U1-Pad19)
- U1 pad 28: col3 -> col5
- U1 pad 29: col4 -> col3
- U1 pad 30: col5 -> Net-(U1-Pad30)
- U1 pad 32: col6 -> Net-(U1-Pad32)
- U1 pad 36: row3 -> Net-(U1-Pad36)
- U1 pad 37: row2 -> Net-(U1-Pad37)
- U1 pad 8: col7 -> Net-(U1-Pad8)
- U1 pad 9: col8 -> Net-(U1-Pad9)
Routing:
- net col0: track 0.00 -> 162.0 mm, vias 0 -> 1
- net col11: track 0.00 -> 152.4 mm
- net col2: track 0.00 -> 148.4 mm, vias 0 -> 1
- net col1: track 0.00 -> 145.4 mm, vias 0 -> 1
- net col10: track 0.00 -> 135.0 mm
- net col3: track 0.00 -> 131.0 mm, vias 0 -> 1
- net col8: track 0.00 -> 117.4 mm
- net col9: track 0.00 -> 113.1 mm
- net col7: track 0.00 -> 101.3 mm
- net col5: track 0.00 -> 79.9 mm, vias 0 -> 1
- net col6: track 0.00 -> 74.2 mm
- net row0: track 200.4 -> 273.0 mm
- net col4: track 0.00 -> 69.3 mm
- net row2: track 200.2 -> 250.3 mm
- net +5V: track 0.00 -> 15.2 mm
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Other:
- net class class1: clearance 0.4 -> 0.2; trace_width 0.5 -> 0.45

Commit message: re 	Routing
Parts:
- moved C7 17.9 mm to (144.5, 65.9), turned to 0 degrees
- moved C1 14.2 mm to (162.7, 78.6)
- moved C2 14.2 mm to (162.7, 69.1)
- moved Y1 14.2 mm to (162.7, 73.8)
- moved C3 8.65 mm to (152.2, 65.9)
- moved C5 8.21 mm to (162.7, 64.9), turned to 270 degrees
- moved SW1 7.39 mm to (162.7, 49.2), turned to 90 degrees
- moved R4 7.14 mm to (147.6, 86.5), turned to 180 degrees
- moved C4 6.35 mm to (153.2, 86.5), turned to 0 degrees
- moved R1 4.63 mm to (162.7, 57.1), turned to 270 degrees
- moved F1 3.60 mm to (141.3, 57.2)
- moved C6 1.82 mm to (140.5, 71.4), turned to 270 degrees
- moved R2 0.79 mm to (150.8, 57.1)
- moved R3 0.16 mm to (147.6, 57.1)
- turned U1 to 270 degrees
Routing:
- net GND: track 15.9 -> 108.2 mm, vias 0 -> 2
- net +5V: track 15.2 -> 87.5 mm, vias 0 -> 6
- net col4: track 69.3 -> 99.5 mm, vias 0 -> 6
- net row0: track 273.0 -> 249.6 mm, vias 0 -> 2
- net col1: track 145.4 -> 125.0 mm, vias 1 -> 5
- net col0: track 162.0 -> 142.2 mm, vias 1 -> 4
- net col3: track 131.0 -> 114.1 mm, vias 1 -> 6
- net Net-(R1-Pad1): track 6.54 -> 23.1 mm
- net row1: track 203.1 -> 218.7 mm
- net col2: track 148.4 -> 135.0 mm, vias 1 -> 6
- net Net-(C2-Pad1): track 4.72 -> 15.7 mm, vias 0 -> 3
- net Net-(R3-Pad1): track 1.55 -> 11.9 mm
- net Net-(R2-Pad1): track 2.88 -> 12.3 mm
- net col6: track 74.2 -> 81.0 mm, vias 0 -> 7
- net Net-(R4-Pad2): track 0.00 -> 5.46 mm
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
Commit message: before check
Parts:
- moved USB1 0.79 mm to (150.0, 45.2)
Connections:
- U1 pad 10: Net-(U1-Pad10) -> row0
- U1 pad 11: Net-(U1-Pad11) -> col5
- U1 pad 18: Net-(U1-Pad18) -> col0
- U1 pad 19: Net-(U1-Pad19) -> col1
- U1 pad 20: Net-(U1-Pad20) -> col2
- U1 pad 21: Net-(U1-Pad21) -> col3
- U1 pad 22: Net-(U1-Pad22) -> col4
- U1 pad 25: col0 -> row3
- U1 pad 26: col1 -> row1
- U1 pad 27: col2 -> Net-(U1-Pad27)
- U1 pad 28: col5 -> Net-(U1-Pad28)
- U1 pad 29: col3 -> Net-(U1-Pad29)
- U1 pad 30: Net-(U1-Pad30) -> row2
- U1 pad 36: Net-(U1-Pad36) -> col6
- U1 pad 37: Net-(U1-Pad37) -> col7
- U1 pad 38: Net-(U1-Pad38) -> col8
- U1 pad 39: Net-(U1-Pad39) -> col9
- U1 pad 40: Net-(U1-Pad40) -> col10
- U1 pad 41: Net-(U1-Pad41) -> col11
Routing:
- net row1: track 218.7 -> 254.1 mm, vias 0 -> 3
- net row2: track 250.2 -> 276.3 mm, vias 3 -> 5
- net col11: track 154.7 -> 179.3 mm
- net row3: track 153.5 -> 177.9 mm, vias 0 -> 2
- net col0: track 142.2 -> 166.3 mm, vias 4 -> 0
- net col6: track 81.0 -> 104.9 mm, vias 7 -> 0
- net col7: track 98.3 -> 121.4 mm, vias 8 -> 0
- net col4: track 99.5 -> 120.7 mm, vias 6 -> 1
- net col8: track 118.0 -> 138.8 mm, vias 7 -> 0
- net col1: track 125.0 -> 145.8 mm, vias 5 -> 1
- net col9: track 118.3 -> 138.9 mm, vias 7 -> 0
- net col5: track 75.2 -> 95.6 mm, vias 6 -> 4
- net col3: track 114.1 -> 132.7 mm, vias 6 -> 0
- net col10: track 140.3 -> 158.0 mm, vias 4 -> 0
- net col2: track 135.0 -> 151.8 mm, vias 6 -> 0
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Other:
- net class class1: trace_width 0.45 -> 0.381

Commit message: fix dcr check error and chgenge switch footprint
Parts:
- SW10, SW11, SW12, SW13, SW14, SW15, SW16, SW17, SW18, SW19, SW2, SW20, SW21, SW22, SW23, SW24, SW25, SW26, SW27, SW28, SW29, SW3, SW30, SW31, SW32, SW33, SW34, SW35, SW36, SW37, SW38, SW39, SW4, SW41, SW43, SW44, SW5, SW6, SW7, SW8, SW9: footprint kbd:CherryMX-Hotswap-v2 -> MX_Only:MXOnly-1U-Hotswap
- SW40, SW42: footprint kbd:CherryMX-Hotswap-v2 -> MX_Only:MXOnly-1.5U-Hotswap
- moved R3 0.73 mm to (148.4, 57.2)
- moved SW2 0.07 mm to (270.7, 65.1)
Routing:
- net col11: track 179.3 -> 168.1 mm
- net col1: track 145.8 -> 140.3 mm, vias 1 -> 4
- net Net-(D3-Pad2): track 10.9 -> 5.41 mm
- net Net-(D34-Pad2): track 10.9 -> 5.41 mm
- net Net-(D1-Pad2): track 10.9 -> 5.57 mm
- net col7: track 121.4 -> 116.1 mm, vias 0 -> 6
- net col6: track 104.9 -> 99.7 mm, vias 0 -> 6
- net col0: track 166.3 -> 161.6 mm, vias 0 -> 4
- net Net-(D2-Pad2): track 9.79 -> 5.41 mm
- net col8: track 138.8 -> 134.6 mm, vias 0 -> 6
- net col4: track 120.7 -> 116.9 mm, vias 1 -> 6
- net Net-(D5-Pad2): track 7.70 -> 4.39 mm
- net Net-(D39-Pad2): track 7.72 -> 4.42 mm
- net Net-(D38-Pad2): track 7.72 -> 4.42 mm
- net Net-(D29-Pad2): track 7.70 -> 4.39 mm
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- added copper zone on B.Cu, net (none)
Other:
- board text added: "psykbd V1.0 PCB Desgine by psychobmx"
